File: analog_output_circuit/tl071.sch (KiCad schematic (older format))
At the start: 10 parts, among them J1 Analog input, J2 Analog output, U1 TL071

Commit message: analog output kicad updates
Parts:
- J1, J2, J?: symbol Screw_Terminal_01x02 -> tl071-rescue:Screw_Terminal_01x02
- R1, R2, R3, R4, R? (x2): symbol R -> tl071-rescue:R
- U1: symbol TL071 -> tl071-rescue:TL071
Connections:
- wire segments 36 -> 44
Changed lines of the file:
@@
-EESchema Schematic File Version 2
-LIBS:power
-LIBS:device
-LIBS:switches
-LIBS:relays
-LIBS:motors
-LIBS:transistors
-LIBS:conn
-LIBS:linear
-LIBS:regul
-LIBS:74xx
-LIBS:cmos4000
-LIBS:adc-dac
-LIBS:memory
-LIBS:xilinx
-LIBS:microcontrollers
-LIBS:dsp
-LIBS:microchip
-LIBS:analog_switches
-LIBS:motorola
-LIBS:texas
-LIBS:intel
-LIBS:audio
-LIBS:interface
-LIBS:digital-audio
-LIBS:philips
-LIBS:display
-LIBS:cypress
-LIBS:siliconi
-LIBS:opto
-LIBS:atmel
-LIBS:contrib
-LIBS:valves
-EELAYER 25 0
+EESchema Schematic File Version 4
+LIBS:tl071-cache
+EELAYER 26 0
 EELAYER END
 $Descr A4 11693 8268
@@
 $EndDescr
 $Comp
-L TL071 U1
+L tl071-rescue:TL071 U1
 U 1 1 5AE3572D
 P 4800 3250
@@
 $EndComp
 $Comp
-L Screw_Terminal_01x02 J1
+L tl071-rescue:Screw_Terminal_01x02 J1
 U 1 1 5AE357AE
 P 5250 4700
@@
 $EndComp
 $Comp
-L R R3
+L tl071-rescue:R R3
 U 1 1 5AE35831
 P 3500 4700
@@
 $EndComp
 $Comp
-L R R4
+L tl071-rescue:R R4
 U 1 1 5AE3590B
 P 4250 4700
@@
 $EndComp
 $Comp
-L Screw_Terminal_01x02 J2
+L tl071-rescue:Screw_Terminal_01x02 J2
 U 1 1 5AE35979
 P 6050 3450
@@
 $EndComp
 $Comp
-L R R1
+L tl071-rescue:R R1
 U 1 1 5AE35B50
 P 2000 3350
@@
 $EndComp
 $Comp
-L R R2
+L tl071-rescue:R R2
 U 1 1 5AE35C00
 P 2000 3900
@@
 	3150 2350 3150 3600
 Wire Wire Line
-	2000 3500 2000 3750
+	2000 3500 2000 3600
 Wire Wire Line
 	2750 3600 2750 3150
@@
 	4850 4800 5050 4800
 Wire Wire Line
-	3350 3650 5400 3650
+	3350 3650 4800 3650
 Wire Wire Line
 	4800 3650 4800 3550
 Wire Wire Line
-	3650 4700 4100 4700
+	3650 4700 3900 4700
 Wire Wire Line
 	3900 4700 3900 3350
@@
 	4700 3600 4700 3550
 Wire Wire Line
-	1750 2950 4700 2950
+	1750 2950 2000 2950
 Connection ~ 2000 2950
 Wire Wire Line
@@
 NoConn ~ 5100 3250
 $Comp
-L R R?
+L tl071-rescue:R R?
 U 1 1 5AE4A828
 P 2300 2350
@@
 $EndComp
 $Comp
-L R R?
+L tl071-rescue:R R?
 U 1 1 5AE4A89F
 P 3000 2350
@@
 $EndComp
 Wire Wire Line
-	2450 2350 2850 2350
+	2450 2350 2600 2350
 Connection ~ 2600 2350
 $Comp
-L GND #PWR?
+L power:GND #PWR?
 U 1 1 5AE4AACE
 P 3800 2450
@@
 $EndComp
 $Comp
-L +12V #PWR?
+L power:+12V #PWR?
 U 1 1 5AE4ABF9
 P 1650 2550
@@
 $EndComp
 Wire Wire Line
-	3800 2200 3800 2450
+	3800 2200 3800 2350
 Wire Wire Line
 	3800 2350 3150 2350
@@
 	2150 2350 2000 2350
 Wire Wire Line
-	2000 1750 2000 2950
+	2000 1750 2000 2350
 Wire Wire Line
 	1650 2550 2000 2550
 Connection ~ 2000 2550
 $Comp
-L Screw_Terminal_01x02 J?
+L tl071-rescue:Screw_Terminal_01x02 J?
 U 1 1 5AE4ADC2
 P 3250 1750
@@
 	2900 2200 3800 2200
 Connection ~ 3800 2350
+Wire Wire Line
+	2000 3600 2000 3750
+Wire Wire Line
+	3900 4700 4100 4700
+Wire Wire Line
+	4800 3650 5400 3650
+Wire Wire Line
+	2000 2950 4700 2950
+Wire Wire Line
+	2600 2350 2850 2350
+Wire Wire Line
+	2000 2550 2000 2950
+Wire Wire Line
+	2000 2350 2000 2550
+Wire Wire Line
+	3800 2350 3800 2450
 $EndSCHEMATC
